File: Board.sch (EAGLE design)
At the start: 29 parts, among them Q1 N-MOS-FET, Q2 N-MOS-FET, Q3 N-MOS-FET, U2 STM32F07

Commit message: switched n-mos to p-mos for common cathode RGBs
Parts:
- removed Q1, Q2, Q3: N-MOS-FET, YabzLib:N-MOS-FET
- removed SWITCH: (no value), pinhead:PINHD-1X2
- added OUT-SWITCH: (no value), pinhead:PINHD-1X2
- added R13, R14, R15: 250, rcl:R-US_R0603
- added U$10, U$11, U$9: P-MOS-FET, YabzLib:P-MOS-FET
- renumbered BARREL to PWR-INPUT
Connections:
- new net N$6: R7.2, SV1.1
- new net N$7: R13.1, U$9.G
- new net N$8: R14.1, U$10.G
- net +3V3: now also U$10.S, U$11.S, U$9.S; no longer SV1.1
- net GND: now also SV1.4; no longer Q1.S, Q2.S, Q3.S
- net LED-B: now also R15.2; no longer Q3.G
- net LED-G: now also R14.2; no longer Q2.G
- net LED-R: now also R13.2; no longer Q1.G
- net N$1: now also OUT-SWITCH.2; no longer PWR-SWITCH.2
- net N$11: now also R15.1, U$11.G; no longer R6.1, SV1.3
- net N$12: now also R5.1, U$9.D; no longer R7.1, SV1.4
- net N$13: now also R6.1, U$10.D; no longer Q2.D, R6.2
- net N$15: now also R7.1, U$11.D; no longer Q1.D, R5.2
- net N$2: now also R5.2, SV1.3; no longer R5.1, SV1.2
- net N$5: now also R6.2, SV1.2; no longer Q3.D, R7.2
- net VBAT: now also PWR-SWITCH.2; no longer SWITCH.2
- net VIN: now also OUT-SWITCH.1; no longer SWITCH.1
Other:
- moved on the sheet: PWR-SWITCH, R5, R6, R7, SV1
